Commit message: fix: replaced local path to global

File: urdf/bot_mecanum.urdf (robot description, URDF)
Before this commit: robot bot, 9 links, 8 joints
Links:
- link front_left_wheel: geometry collision sphere radius=.1; visual mesh filename=package://snowbot123/meshes/mecanum_wheel_left.STL scale=0.002 .002 0.002
- link front_right_wheel: geometry collision sphere radius=.1; visual mesh filename=package://snowbot123/meshes/mecanum_wheel_right.STL scale=0.002 .002 0.002
- link rear_left_wheel: geometry collision sphere radius=.1; visual mesh filename=package://snowbot123/meshes/mecanum_wheel_right.STL scale=0.002 .002 0.002
- link rear_right_wheel: geometry collision sphere radius=.1; visual mesh filename=package://snowbot123/meshes/mecanum_wheel_left.STL scale=0.002 .002 0.002
